Commit message: gazebo visual success

File: urdf/serial_t800.urdf (robot description, URDF)
Before this commit: robot t800, 30 links, 29 joints
Links:
- link LINK_HIP_PITCH_R: geometry collision sphere radius=0.07; visual mesh filename=package://t800_description/meshes/LINK_HIP_PITCH_L.dae
- link LINK_SHOULDER_PITCH_R: geometry collision sphere radius=0.06; visual mesh filename=package://t800_description/meshes/LINK_SHOULDER_PITCH_L.dae
- link LINK_SHOULDER_ROLL_R: geometry visual mesh filename=package://t800_description/meshes/LINK_SHOULDER_ROLL_L.dae
