Commit message: world setup done

File: urdf/serial_t800_visual_mid360_imu_upper_collision.urdf (robot description, URDF)
Before this commit: robot t800, 32 links, 31 joints
Joints:
- joint t800_chest_to_mid360: origin xyz=0.13 0.0 0.38 rpy=0.0 -0.0 0 -> xyz=0.13 0.0 0.38 rpy=0.0 0.3489 0

Commit message: no big change

File: urdf/serial_t800_visual_mid360_imu_upper_collision.urdf (robot description, URDF)
Before this commit: robot t800, 32 links, 31 joints
Joints:
- joint t800_chest_to_mid360: origin xyz=0.13 0.0 0.38 rpy=0.0 0.3489 0 -> xyz=0.13 0.0 0.38 rpy=0.0 0.8722 0
