Commit message: sim mid360 with t800 success

File: urdf/old/serial_t800.urdf (robot description, URDF)
Before this commit: robot t800, 30 links, 29 joints
Links:
- link LINK_ELBOW_PITCH_R: geometry collision sphere radius=0.05; visual mesh filename=package://t800_description/meshes/LINK_ELBOW_PITCH_R.obj
